File: led_20w.kicad_sch (KiCad schematic)
At the start: 22 parts

Commit message: 60W gbr 3d pdf
Parts:
- added LED11, LED12, LED13, LED14, LED17, LED18, LED19, LED20, LED21, LED24, LED25, LED26, LED27, LED28, LED31, LED32, LED33, LED34, LED35, LED38, LED39, LED40, LED41, LED42, LED45, LED46, LED47, LED48, LED49, LED50, LED51, LED52, LED53, LED54, LED55, LED56, LED57, LED58, LED59, LED60: JB2835BWT-G-H40EA0000-N0000001, 2835-library:JB2835BWTGH40EA0000N0000001, symbol 2835 LED SMD:JB2835BWT-G-H40EA0000-N0000001
- gave numbers to parts that had none: 6
Connections:
- net +24V: now also LED11.2, LED13.2, LED17.2, LED18.2, LED21.2, LED24.2, LED27.2, LED31.2, LED33.2, LED35.2, LED39.2, LED41.2, LED45.2, LED46.2, LED49.2, LED50.2, LED53.2, LED55.2, LED57.2, LED59.2
- net GND: now also LED23.1, LED44.1, LED12.1, LED14.1, LED19.1, LED20.1, LED25.1, LED26.1, LED28.1, LED32.1, LED34.1, LED38.1, LED40.1, LED42.1, LED47.1, LED48.1, LED51.1, LED52.1, LED54.1, LED56.1, LED58.1, LED60.1; no longer LED23.2, LED44.2
- net at LED22.1: now also LED23.2; no longer LED23.1
- net at LED43.1: now also LED44.2; no longer LED44.1
- new net: LED31.1, LED32.2
- new net: LED59.1, LED60.2
- new net: LED11.1, LED12.2
- new net: LED41.1, LED42.2
- new net: LED21.1, LED25.2
- new net: LED35.1, LED38.2
- new net: LED57.1, LED58.2
- new net: LED55.1, LED56.2
- new net: LED46.1, LED48.2
- new net: LED17.1, LED19.2
- new net: LED39.1, LED40.2
- new net: LED50.1, LED52.2
- new net: LED18.1, LED20.2
- new net: LED24.1, LED26.2
- new net: LED33.1, LED34.2
- new net: LED27.1, LED28.2
- new net: LED13.1, LED14.2
- new net: LED45.1, LED47.2
- new net: LED49.1, LED51.2
- new net: LED53.1, LED54.2
Other:
- note added: "( (2 SERIES )*10 ) * 3 BLOCK"
- note removed: "(2 SERIES )*10 LED PANEL"
- moved on the sheet: LED1, LED10, LED15, LED16, LED2, LED22, LED23, LED29, LED3, LED30, LED36, LED37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
